Commit message: Add collisions to backbone urdf.

File: urdf/backbone_manipulator.urdf (robot description, URDF)
Before this commit: robot backbone_manipulator, 12 links, 11 joints
Links:
- link base: geometry collision sphere radius=0.1; visual sphere radius=0.1
- link robot0: geometry collision sphere radius=0.1; visual sphere radius=0.1
- link robot1: geometry collision sphere radius=0.1; visual sphere radius=0.1
- link robot2: geometry collision sphere radius=0.1; visual sphere radius=0.1
- link robot3: geometry collision sphere radius=0.1; visual sphere radius=0.1
- link robot4: geometry collision sphere radius=0.1; visual sphere radius=0.1
Joints:
- joint base_to_network: axis 1.0 0 0 -> 0 1.0 0
- joint baselink_to_base: axis 0 0 1.0 -> 1.0 0 0
- joint network_to_robot0: axis 0 0 1.0 -> 1.0 0 0
- joint network_to_robot1: axis 0 0 1.0 -> 1.0 0 0
- joint network_to_robot2: axis 0 0 1.0 -> 1.0 0 0
- joint network_to_robot3: axis 0 0 1.0 -> 1.0 0 0
- joint network_to_robot4: axis 0 0 1.0 -> 1.0 0 0
- joint robot1_to_network: axis 1.0 0 0 -> 0 1.0 0
- joint robot2_to_network: axis 1.0 0 0 -> 0 1.0 0
- joint robot3_to_network: axis 1.0 0 0 -> 0 1.0 0
- joint robot4_to_network: axis 1.0 0 0 -> 0 1.0 0
