Commit message: Update manipulator URDF.
- Continuous joints were replaced by revolute joints;
- End effectors's parent joint is now fixed;
- Added missing collision geometry.

File: urdf/backbone.urdf (robot description, URDF)
Before this commit: robot backbone_manipulator, 12 links, 11 joints
Links:
- link base_link: geometry collision cylinder length=0.01 radius=0.05; visual cylinder length=0.01 radius=0.05
- link network_base_to_robot4: geometry collision cylinder length=5 radius=0.005; visual cylinder length=5 radius=0.005
- link network_robot1_to_robot0: geometry collision cylinder length=5 radius=0.005; visual cylinder length=5 radius=0.005
- link network_robot2_to_robot1: geometry collision cylinder length=5 radius=0.005; visual cylinder length=5 radius=0.005
- link network_robot3_to_robot2: geometry collision cylinder length=5 radius=0.005; visual cylinder length=5 radius=0.005
- link network_robot4_to_robot3: geometry collision cylinder length=5 radius=0.005; visual cylinder length=5 radius=0.005
Joints:
- joint baselink_to_base: limit (none) -> lower=-1.5708 upper=1.5708 effort=30 velocity=1.0; type continuous -> revolute
- joint network_to_robot0: axis 0 0 1.0 -> (none); type continuous -> fixed
- joint network_to_robot1: limit (none) -> lower=-1.5708 upper=1.5708 effort=30 velocity=1.0; type continuous -> revolute
- joint network_to_robot2: limit (none) -> lower=-1.5708 upper=1.5708 effort=30 velocity=1.0; type continuous -> revolute
- joint network_to_robot3: limit (none) -> lower=-1.5708 upper=1.5708 effort=30 velocity=1.0; type continuous -> revolute
- joint network_to_robot4: limit (none) -> lower=-1.5708 upper=1.5708 effort=30 velocity=1.0; type continuous -> revolute

Commit message: Remove constraints in backbone URDF.

File: urdf/backbone.urdf (robot description, URDF)
Before this commit: robot backbone_manipulator, 12 links, 11 joints
Joints:
- joint base_to_network: limit lower=-1.5708 upper=1.5708 effort=30 velocity=1.0 -> lower=-1.5708 upper=1.5708 effort=1000 velocity=100.0
- joint baselink_to_base: limit lower=-1.5708 upper=1.5708 effort=30 velocity=1.0 -> lower=-1.5708 upper=1.5708 effort=1000 velocity=100.0
- joint network_to_robot1: limit lower=-1.5708 upper=1.5708 effort=30 velocity=1.0 -> lower=-1.5708 upper=1.5708 effort=1000 velocity=100.0
- joint network_to_robot2: limit lower=-1.5708 upper=1.5708 effort=30 velocity=1.0 -> lower=-1.5708 upper=1.5708 effort=1000 velocity=100.0
- joint network_to_robot3: limit lower=-1.5708 upper=1.5708 effort=30 velocity=1.0 -> lower=-1.5708 upper=1.5708 effort=1000 velocity=100.0
- joint network_to_robot4: limit lower=-1.5708 upper=1.5708 effort=30 velocity=1.0 -> lower=-1.5708 upper=1.5708 effort=1000 velocity=100.0
- joint robot1_to_network: limit lower=-1.5708 upper=1.5708 effort=30 velocity=1.0 -> lower=-1.5708 upper=1.5708 effort=1000 velocity=100.0
- joint robot2_to_network: limit lower=-1.5708 upper=1.5708 effort=30 velocity=1.0 -> lower=-1.5708 upper=1.5708 effort=1000 velocity=100.0
- joint robot3_to_network: limit lower=-1.5708 upper=1.5708 effort=30 velocity=1.0 -> lower=-1.5708 upper=1.5708 effort=1000 velocity=100.0
- joint robot4_to_network: limit lower=-1.5708 upper=1.5708 effort=30 velocity=1.0 -> lower=-1.5708 upper=1.5708 effort=1000 velocity=100.0
